File: RGB_sorter/RGB_sorter.kicad_sch (KiCad schematic)
At the start: 32 parts, among them J1 Conn_01x03_Pin, J2 Conn_01x03_Pin, J3 Conn_01x02_Pin, J4 Conn_01x02_Pin, J5 Screw_Terminal_01x03, J6 Conn_01x04_Pin, U1 L298N, U2 L7805, U3 ULN2003

Commit message: PCB Uredjaj za sortiranje boja
PCB edit
Parts:
- removed C3: 10uF, symbol Device:C_Polarized_Small_US
- removed C4: 1uF, symbol Device:C_Polarized_Small_US
- removed C5: 0.1uF, symbol Device:C_Polarized_Small_US
- removed D1, D2, D3, D4, D5, D6, D7, D8: 1N4001, Diode_THT:D_DO-41_SOD81_P10.16mm_Horizontal, symbol Diode:1N4001
- removed J2: Conn_01x03_Pin, symbol Connector:Conn_01x03_Pin
- removed J3, J4: Conn_01x02_Pin, symbol Connector:Conn_01x02_Pin
- removed J5: Screw_Terminal_01x03, symbol Connector:Screw_Terminal_01x03
- added BZ1: Buzzer, Buzzer_Beeper:Buzzer_12x9.5RM7.6, symbol Device:Buzzer
- added C3, C6: 10uF, Capacitor_SMD:C_1206_3216Metric, symbol Device:C_Small
- added C4: 1uF, Capacitor_SMD:C_0805_2012Metric, symbol Device:C_Small
- added C5: 0.1uF, Capacitor_SMD:C_0805_2012Metric, symbol Device:C_Small
- added D1, D2, D3, D4, D5, D6, D7, D8: SS110, Diode_SMD:D_SMA, symbol Diode:SS110
- added D14: LED_Red, LED_THT:LED_D5.0mm, symbol Device:LED_Small_Filled
- added D15: LED_Green, LED_THT:LED_D5.0mm, symbol Device:LED_Small_Filled
- added D16: LED_Blue, LED_THT:LED_D5.0mm, symbol Device:LED_Small_Filled
- added J10: TCS34725, Connector_PinHeader_2.54mm:PinHeader_1x04_P2.54mm_Vertical, symbol Connector:Conn_01x04_Pin
- added J11: IR sensor, Connector_PinHeader_2.54mm:PinHeader_1x03_P2.54mm_Vertical, symbol Connector:Conn_01x03_Pin
- added J2: Power, TerminalBlock_Phoenix:TerminalBlock_Phoenix_MKDS-1,5-2-5.08_1x02_P5.08mm_Horizontal, symbol Connector:Screw_Terminal_01x02
- added J3: Motor A, TerminalBlock_Phoenix:TerminalBlock_Phoenix_MKDS-1,5-2-5.08_1x02_P5.08mm_Horizontal, symbol Connector:Screw_Terminal_01x02
- added J4: Motor B, TerminalBlock_Phoenix:TerminalBlock_Phoenix_MKDS-1,5-2-5.08_1x02_P5.08mm_Horizontal, symbol Connector:Screw_Terminal_01x02
- added J8: Conn_01x05_Pin, Connector_JST:JST_XH_B5B-XH-A_1x05_P2.50mm_Vertical, symbol Connector:Conn_01x05_Pin
- added JP1, JP2, JP3: ~, Connector_PinHeader_2.54mm:PinHeader_1x02_P2.54mm_Vertical, symbol Jumper:Jumper_2_Small_Open
- added R6, R7, R8, R9: 220, Resistor_SMD:R_0805_2012Metric, symbol Device:R_Small
- added SW1: START, Button_Switch_THT:SW_PUSH-12mm_Wuerth-430476085716, symbol Switch:SW_SPST
- added SW2: RESET, Button_Switch_THT:SW_PUSH-12mm_Wuerth-430476085716, symbol Switch:SW_SPST
- added SW3: STOP, Button_Switch_THT:SW_PUSH-12mm_Wuerth-430476085716, symbol Switch:SW_SPST
- added U4: NUCLEO64-F411RE, custom_footprints:MODULE_NUCLEO-F446RE, symbol MCU_Module:NUCLEO64-F411RE
- C1: footprint (none) -> Capacitor_SMD:CP_Elec_8x10.5
- C2: footprint (none) -> Capacitor_SMD:CP_Elec_10x10.5
- D10, D11, D12, D13: footprint (none) -> LED_SMD:LED_1206_3216Metric
- D9: footprint (none) -> LED_SMD:LED_0805_2012Metric
- J1: value Conn_01x03_Pin -> Servo; footprint (none) -> Connector_PinHeader_2.54mm:PinHeader_1x03_P2.54mm_Vertical
- J6: value Conn_01x04_Pin -> LCD; footprint (none) -> Connector_PinHeader_2.54mm:PinHeader_1x04_P2.54mm_Vertical
- R1: footprint (none) -> Resistor_SMD:R_0805_2012Metric
- R2, R3, R4, R5: value 1k -> 470; footprint (none) -> Resistor_SMD:R_0805_2012Metric
- U1: footprint Package_TO_SOT_THT:TO-220-15_P2.54x5.08mm_StaggerOdd_Lead4.58mm_Vertical -> custom_footprints:L298n
- U2: footprint (none) -> Package_TO_SOT_SMD:TO-252-2
- U3: footprint (none) -> Package_SO:SOIC-16_3.9x9.9mm_P1.27mm
Connections:
- net +12V: now also U3.9 (COM), C3.1, C6.1, D1.1 (K), D2.1 (K), D3.1 (K), D4.1 (K), J2.1 (Pin_1), JP3.1 (A)
- net +5V: now also J1.2 (Pin_2), C4.1, C5.1, JP1.1 (A), JP2.1 (A), U4.6 (E5V)
- net GND: now also C1.2, J1.3 (Pin_3), J6.1 (Pin_1), U1.15 (SENSE_B), BZ1.2 (-), C3.2, C4.2, C5.2, C6.2, D14.1 (K), D15.1 (K), D16.1 (K), D5.2 (A), D6.2 (A), D7.2 (A), D8.2 (A), J10.3 (Pin_3), J11.3 (Pin_3), J2.2 (Pin_2), SW1.2 (B), SW2.2 (B), SW3.2 (B), U4.19 (GND), U4.20 (GND), U4.22 (GND), U4.47 (GND), U4.58 (GND), U4.8 (GND)
- net at U1.14 (OUT4): now also D4.2 (A), D8.1 (K), J4.2 (Pin_2)
- net at R5.1: now also R2.1, R3.1, R4.1, J8.1 (Pin_1), JP3.2 (B)
- net at U1.13 (OUT3): now also D3.2 (A), D7.1 (K), J4.1 (Pin_1)
- net at U1.3 (OUT2): now also D2.2 (A), D6.1 (K), J3.2 (Pin_2)
- net at D13.1 (K): now also U3.13 (O4), J8.5 (Pin_5)
- net at U1.2 (OUT1): now also D1.2 (A), D5.1 (K), J3.1 (Pin_1)
- net at D11.1 (K): now also U3.15 (O2), J8.3 (Pin_3)
- net I1: now reaches U3.1 (I1)
- net I1: now also U4.32 (PA4); no longer J6.1 (Pin_1)
- net at U3.14 (O3): now also D12.1 (K), J8.4 (Pin_4)
- net at U3.16 (O1): now also D10.1 (K), J8.2 (Pin_2)
- net at J6.2 (Pin_2): now also U4.18 (+5V); no longer U3.2 (I2)
- net I3: now reaches U3.3 (I3)
- net I3: now also U4.53 (PA7); no longer J6.3 (Pin_3)
- net I4: now reaches U3.4 (I4)
- net I4: now also U4.59 (PA9); no longer J6.4 (Pin_4)
- net IN3: now reaches U1.10 (IN3)
- net IN3: now also U4.63 (PB10)
- net IN4: now reaches U1.12 (IN4)
- net IN4: now also U4.60 (PB2)
- net at U1.11 (EnB): now also JP2.2 (B)
- net IN1: now reaches U1.5 (IN1)
- net IN1: now also U4.17 (PA15); no longer J1.1 (Pin_1)
- net at U1.6 (EnA): now also JP1.2 (B); no longer J1.3 (Pin_3)
- net IN2: now reaches U1.7 (IN2)
- net IN2: now also U4.30 (PA1); no longer J1.2 (Pin_2)
- new net: J10.1 (Pin_1), U4.41 (PB8)
- new net: J10.2 (Pin_2), U4.43 (PB9)
- new net: R7.1, U4.40 (PC8)
- new net: D15.2 (A), R7.2
- new net: R8.1, U4.1 (PC10)
- new net: D16.2 (A), R8.2
- new net: R6.1, U4.2 (PC11)
- new net: R9.1, U4.42 (PC6)
- new net: J11.1 (Pin_1), U4.57 (PC7)
- new net: SW1.1 (A), U4.64 (PB15)
- new net: SW3.1 (A), U4.66 (PB14)
- new net: SW2.1 (A), U4.68 (PB13)
- new net: BZ1.1 (+), R9.2
- new net: D14.2 (A), R6.2
- new net +3V3: J10.4 (Pin_4), J11.2 (Pin_2), U4.16 (+3V3)
- new net I2: U3.2 (I2), U4.51 (PA6)
- new net PA8: J6.3 (Pin_3), U4.61 (PA8)
- new net PB4: J1.1 (Pin_1), U4.65 (PB4)
- new net PC9: J6.4 (Pin_4), U4.39 (PC9)
- no-connect marks 0 -> 44
Other:
- company: (none) -> Tehnicko veleuciliste u Zagrebu
- title: (none) -> Uredjaj za sortiranje boja
- moved on the sheet: C1, C2, D10, D11, D12, D13, D9, R1, R2, R3, R4, R5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

Commit message: Upgrade PCB-a
Shematic i PCB edit
Parts:
- removed J10: TCS34725, Connector_PinHeader_2.54mm:PinHeader_1x04_P2.54mm_Vertical, symbol Connector:Conn_01x04_Pin
- removed SW1: START, Button_Switch_THT:SW_PUSH-12mm_Wuerth-430476085716, symbol Switch:SW_SPST
- removed SW2: RESET, Button_Switch_THT:SW_PUSH-12mm_Wuerth-430476085716, symbol Switch:SW_SPST
- removed SW3: STOP, Button_Switch_THT:SW_PUSH-12mm_Wuerth-430476085716, symbol Switch:SW_SPST
- added J5: TCS34725, Connector_PinHeader_2.54mm:PinHeader_1x06_P2.54mm_Vertical, symbol Connector:Conn_01x06_Pin
- added J7: IR sensor2, Connector_PinHeader_2.54mm:PinHeader_1x03_P2.54mm_Vertical, symbol Connector:Conn_01x03_Pin
- added SW1: START, Button_Switch_THT:SW_PUSH-12mm_Wuerth-430476085716, symbol Switch:SW_Push
- added SW2: RESET, Button_Switch_THT:SW_PUSH-12mm_Wuerth-430476085716, symbol Switch:SW_Push
- added SW3: STOP, Button_Switch_THT:SW_PUSH-12mm_Wuerth-430476085716, symbol Switch:SW_Push
- D16: value LED_Blue -> LED_Orange
- J11: value IR sensor -> IR sensor1
Connections:
- net +5V: now also J6.2 (Pin_2)
- net GND: now also J11.2 (Pin_2), J5.2 (Pin_2), J7.2 (Pin_2), SW1.2, SW2.2, SW3.2; no longer J11.3 (Pin_3)
- net I1: now also U4.17 (PA15); no longer U4.32 (PA4)
- net I2: now also U4.3 (PC12); no longer U4.51 (PA6)
- net I3: now also U4.1 (PC10); no longer U4.53 (PA7)
- net I4: now also U4.2 (PC11); no longer U4.59 (PA9)
- net IN1: now also U4.28 (PA0); no longer U4.17 (PA15)
- net IN3: now also U4.65 (PB4); no longer U4.63 (PB10)
- net IN4: now also U4.63 (PB10); no longer U4.60 (PB2)
- net TCS_SCL: now reaches U4.41 (PB8)
- net TCS_SCL: now also J5.4 (Pin_4)
- net TCS_SDA: now reaches U4.43 (PB9)
- net TCS_SDA: now also J5.3 (Pin_3)
- net at U4.40 (PC8): no longer R7.1
- net ORANGE: now reaches R8.1
- net ORANGE: now also U4.36 (PC1); no longer U4.1 (PC10)
- net at U4.18 (+5V): no longer J6.2 (Pin_2)
- net RED: now reaches R6.1
- net RED: now also U4.34 (PB0); no longer U4.2 (PC11)
- net SERVO_PWM: now reaches U4.21 (PB7)
- net SERVO_PWM: now also J1.1 (Pin_1)
- net BUZZER: now reaches U4.37 (PC3)
- net BUZZER: now also R9.1
- net GREEN: now reaches U4.38 (PC0)
- net GREEN: now also R7.1
- net LED: now reaches U4.42 (PC6)
- net LED: now also J5.6 (Pin_6); no longer R9.1
- net INT: now reaches U4.44 (PC5)
- net INT: now also J5.5 (Pin_5)
- net IR_OUT: now reaches J11.1 (Pin_1), U4.57 (PC7)
- net START: now reaches U4.64 (PB15)
- net START: now also SW1.1
- net RESET: now reaches U4.66 (PB14)
- net RESET: now also SW2.1
- net STOP: now reaches U4.68 (PB13)
- net STOP: now also SW3.1
- net IR2_OUT: now reaches U4.72 (PC4)
- net IR2_OUT: now also J7.1 (Pin_1)
- net +3V3 renamed +3.3V
- net +3.3V: now also J11.3 (Pin_3), J5.1 (Pin_1), J7.3 (Pin_3); no longer J11.2 (Pin_2)
- net PA8 renamed LCD_SCL
- removed net PB4: J1.1 (Pin_1), U4.65 (PB4)
- net PC9 renamed LCD_SDA
- no-connect marks 44 -> 42
Other:
- note added: "Indikatori"
- note added: "Konektori"
- note added: "L298N"
- note added: "L7805 5V regulator"
- note added: "STM32F446RET6"
- note added: "Tipkala"
- note added: "ULN2003"
- moved on the sheet: BZ1, C1, C2, C3, C4, C5, C6, D1, D10, D11, D12, D13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
